File: pcb/metrodisplay.kicad_pcb (KiCad board)
At the start: 2 copper layers, 4 parts, among them J1 USB_C_Receptacle_PowerOnly_6P, J2 Conn_02x08_Counter_Clockwise, SW1 SW_Push, U1 ESP32-DEVKITC

Commit message: PCB Routing test
Parts:
- added C1: C_Polarized, Capacitor_THT:CP_Radial_D16.0mm_P7.50mm, F.Cu at (95.3, 26.2)
- added C10: C, easyeda2kicad:C1206, F.Cu at (96.3, 74.5)
- added C11: C, easyeda2kicad:C1206, F.Cu at (99.7, 76.9)
- added C12: C, easyeda2kicad:C1206, F.Cu at (94.5, 76.9)
- added C13: C, easyeda2kicad:C1206, F.Cu at (101.4, 74.5)
- added C14: C, easyeda2kicad:C1206, F.Cu at (91.1, 74.5)
- added C15: C, easyeda2kicad:C1206, F.Cu at (106.5, 74.5)
- added C16: C, easyeda2kicad:C1206, F.Cu at (89.4, 76.9)
- added C17: C, easyeda2kicad:C1206, F.Cu at (104.8, 76.9)
- added C18: RVT470UF35V67RV0056, easyeda2kicad:CAP-SMD_BD10.0-L10.3-W10.3-LS11.0-FD, F.Cu at (29.1, 41.1)
- added C2: C, easyeda2kicad:C1206, F.Cu at (99.7, 86.5)
- added C3: C, easyeda2kicad:C1206, F.Cu at (101.4, 88.8)
- added C4: C, easyeda2kicad:C1206, F.Cu at (104.8, 86.5)
- added C5: C, easyeda2kicad:C1206, F.Cu at (106.5, 88.8)
- added C6: C, easyeda2kicad:C1206, F.Cu at (96.3, 88.8)
- added C7: C, easyeda2kicad:C1206, F.Cu at (94.5, 86.5)
- added C8: C, easyeda2kicad:C1206, F.Cu at (91.1, 88.8)
- added C9: C, easyeda2kicad:C1206, F.Cu at (89.4, 86.5)
- added D1: IR26-21C_L110_TR8, LED_SMD:LED_1206_3216Metric, F.Cu at (29.6, 82.9)
- added J3: Screw_Terminal_01x02, TerminalBlock_Dinkle:TerminalBlock_Dinkle_DT-55-B01X-02_P10.00mm, F.Cu at (112.4, 27.2)
- added JP1: SolderJumper_2_Open, Jumper:SolderJumper-2_P1.3mm_Open_TrianglePad1.0x1.5mm, F.Cu at (88.4, 57.8)
- added JP10: SolderJumper_2_Open, Jumper:SolderJumper-2_P1.3mm_Open_TrianglePad1.0x1.5mm, F.Cu at (99.4, 112.8)
- added JP11: SolderJumper_2_Open, Jumper:SolderJumper-2_P1.3mm_Open_TrianglePad1.0x1.5mm, F.Cu at (96.0, 112.8)
- added JP12: SolderJumper_2_Open, Jumper:SolderJumper-2_P1.3mm_Open_TrianglePad1.0x1.5mm, F.Cu at (92.5, 112.8)
- added JP13: SolderJumper_2_Open, Jumper:SolderJumper-2_P1.3mm_Open_TrianglePad1.0x1.5mm, F.Cu at (88.9, 112.8)
- added JP14: SolderJumper_2_Open, Jumper:SolderJumper-2_P1.3mm_Open_TrianglePad1.0x1.5mm, F.Cu at (85.4, 112.8)
- added JP15: SolderJumper_3_Open, Jumper:SolderJumper-3_P2.0mm_Open_TrianglePad1.0x1.5mm, F.Cu at (114.1, 82.0)
- added JP16: SolderJumper_3_Open, Jumper:SolderJumper-3_P2.0mm_Open_TrianglePad1.0x1.5mm, F.Cu at (80.3, 81.5)
- added JP2: SolderJumper_2_Open, Jumper:SolderJumper-2_P1.3mm_Open_TrianglePad1.0x1.5mm, F.Cu at (92.0, 57.8)
- added JP3: SolderJumper_2_Open, Jumper:SolderJumper-2_P1.3mm_Open_TrianglePad1.0x1.5mm, F.Cu at (95.5, 57.8)
- added JP4: SolderJumper_2_Open, Jumper:SolderJumper-2_P1.3mm_Open_TrianglePad1.0x1.5mm, F.Cu at (99.1, 57.8)
- added JP5: SolderJumper_2_Open, Jumper:SolderJumper-2_P1.3mm_Open_TrianglePad1.0x1.5mm, F.Cu at (102.6, 57.8)
- added JP6: SolderJumper_2_Open, Jumper:SolderJumper-2_P1.3mm_Open_TrianglePad1.0x1.5mm, F.Cu at (105.7, 57.8)
- added JP7: SolderJumper_2_Open, Jumper:SolderJumper-2_P1.3mm_Open_TrianglePad1.0x1.5mm, F.Cu at (110.1, 112.8)
- added JP8: SolderJumper_2_Open, Jumper:SolderJumper-2_P1.3mm_Open_TrianglePad1.0x1.5mm, F.Cu at (106.5, 112.8)
- added JP9: SolderJumper_2_Open, Jumper:SolderJumper-2_P1.3mm_Open_TrianglePad1.0x1.5mm, F.Cu at (103.0, 112.8)
- added R1: FRC1206J102 TS, easyeda2kicad:R1206, F.Cu at (29.6, 80.4)
- added U3: SN74AHCT245PWR, easyeda2kicad:TSSOP-20_L6.5-W4.4-P0.65-LS6.4-BL, F.Cu at (97.7, 100.8)
- added U4: SN74AHCT245PWR, easyeda2kicad:TSSOP-20_L6.5-W4.4-P0.65-LS6.4-BL, F.Cu at (96.8, 65.5)
- J2: footprint Connector_PinHeader_2.54mm:PinHeader_2x08_P2.54mm_Vertical -> easyeda2kicad:PinHeader_2x08_P2.54mm_Vertical_MD
- moved J1 84.3 mm to (5.05, 52.5)
- moved SW1 56.4 mm to (64.5, 82.4)
- moved J2 10.4 mm to (106.0, 80.4), turned to -90 degrees
- moved U1 10.3 mm to (69.4, 48.7), turned to -90 degrees
Connections:
- net Control renamed CTRL
- J2 pad A: A -> Net-(J2-Pin_5)
- J2 pad B: B -> Net-(J2-Pin_12)
- J2 pad B1: B1 -> Net-(J2-Pin_2)
- J2 pad B2: B2 -> Net-(J2-Pin_4)
- J2 pad C: C -> Net-(J2-Pin_6)
- J2 pad CLK: CLK -> Net-(J2-Pin_7)
- J2 pad D: D -> Net-(J2-Pin_11)
- J2 pad E: E -> Net-(J2-Pin_13)
- J2 pad G1: G1 -> Net-(J2-Pin_16)
- J2 pad G2: G2 -> Net-(J2-Pin_14)
- J2 pad LAT: LAT -> Net-(J2-Pin_10)
- J2 pad OE: OE -> Net-(J2-Pin_8)
- J2 pad R1: R1 -> Net-(J2-Pin_1)
- J2 pad R2: R2 -> Net-(J2-Pin_3)
- U1 pad 26: unconnected-(U1-IO4-Pad26) -> LED
Routing:
- net 5V: track 0.00 -> 107.4 mm
- net GND: track 0.00 -> 83.6 mm
- net G1: track 0.00 -> 64.6 mm
- net G2: track 0.00 -> 61.5 mm
- net OELS: track 0.00 -> 61.2 mm
- net LAT: track 0.00 -> 60.6 mm
- net D: track 0.00 -> 58.9 mm
- net E: track 0.00 -> 58.6 mm
- net B: track 0.00 -> 57.8 mm
- net DIRLS: track 0.00 -> 47.2 mm
- net Net-(J2-Pin_1): track 0.00 -> 21.1 mm
- net Net-(J2-Pin_7): track 0.00 -> 19.5 mm
- net Net-(J2-Pin_8): track 0.00 -> 18.4 mm
- net Net-(J2-Pin_3): track 0.00 -> 18.1 mm
- net Net-(J2-Pin_5): track 0.00 -> 17.2 mm
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
Commit message: PCB routing done
Parts:
- removed JP1, JP10, JP11, JP12, JP13, JP14, JP2, JP3, JP4, JP5, JP6, JP7, JP8, JP9: SolderJumper_2_Open, Jumper:SolderJumper-2_P1.3mm_Open_TrianglePad1.0x1.5mm
- added C19: C, easyeda2kicad:C1206, F.Cu at (75.0, 41.2)
- added C20: C, easyeda2kicad:C1206, F.Cu at (93.4, 59.2)
- moved SW1 62.9 mm to (117.3, 48.2), turned to 90 degrees
- moved JP15 46.1 mm to (93.8, 40.6), turned to 135 degrees
- moved D1 45.0 mm to (42.7, 39.8), turned to 90 degrees
- moved C15 43.0 mm to (84.8, 37.4), turned to -135 degrees
- moved R1 42.0 mm to (40.3, 39.8), turned to 90 degrees
- moved C17 41.5 mm to (85.3, 40.3), turned to -135 degrees
- moved J2 40.9 mm to (89.7, 42.9), turned to -45 degrees
- moved C5 40.5 mm to (97.0, 49.5), turned to 45 degrees
- moved C13 39.1 mm to (81.2, 41.0), turned to -135 degrees
- moved C4 38.9 mm to (94.1, 49.0), turned to 45 degrees
- moved U3 38.3 mm to (96.7, 62.5), turned to 135 degrees
- moved C11 37.6 mm to (81.7, 43.9), turned to -135 degrees
- moved U4 37.4 mm to (71.6, 37.8), turned to 135 degrees
- moved C3 36.6 mm to (93.4, 53.1), turned to 45 degrees
- moved C10 35.2 mm to (77.6, 44.6), turned to 45 degrees
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Connections:
- C15 pad 2: unconnected-(C15-Pad2) -> Net-(J2-Pin_16)
- C17 pad 2: Net-(J2-Pin_16) -> unconnected-(C17-Pad2)
- U3 pad 10: unconnected-(U3-GND-Pad10) -> GND
- U3 pad 11: R1 -> OE
- U3 pad 12: B1 -> CLK
- U3 pad 13: R2 -> C
- U3 pad 14: B2 -> A
- U3 pad 15: A -> B2
- U3 pad 16: C -> R2
- U3 pad 17: CLK -> B1
- U3 pad 18: OE -> R1
- U3 pad 2: Net-(J2-Pin_8) -> Net-(J2-Pin_1)
- U3 pad 3: Net-(J2-Pin_7) -> Net-(J2-Pin_2)
- U3 pad 4: Net-(J2-Pin_6) -> Net-(J2-Pin_3)
- U3 pad 5: Net-(J2-Pin_5) -> Net-(J2-Pin_4)
- U3 pad 6: Net-(J2-Pin_4) -> Net-(J2-Pin_5)
- U3 pad 7: Net-(J2-Pin_3) -> Net-(J2-Pin_6)
- U3 pad 8: Net-(J2-Pin_2) -> Net-(J2-Pin_7)
- U3 pad 9: Net-(J2-Pin_1) -> Net-(J2-Pin_8)
- U4 pad 10: unconnected-(U4-GND-Pad10) -> GND
Routing:
- net 5V: track 107.4 -> 276.4 mm, vias 0 -> 2
- net CTRL: track 0.00 -> 99.0 mm
- net OE: track 0.00 -> 68.7 mm
- net CLK: track 0.00 -> 55.3 mm
- net C: track 0.00 -> 52.9 mm
- net A: track 0.00 -> 48.0 mm
- net G1: track 64.6 -> 17.9 mm
- net B2: track 0.00 -> 45.8 mm
- net R2: track 0.00 -> 41.0 mm
- net G2: track 61.5 -> 22.0 mm
- net B1: track 0.00 -> 33.6 mm
- net E: track 58.6 -> 25.2 mm
- net LED: track 0.00 -> 32.2 mm, vias 0 -> 2
- net R1: track 0.00 -> 31.3 mm
- net GND: track 83.6 -> 53.1 mm, vias 0 -> 25
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- added copper zone on B.Cu, net GND
- added copper zone on F.Cu, net GND
Other:
- board outline added: 99.2 x 52.8 mm

Commit message: PCB done
Parts:
- moved JP15 1.77 mm to (95.0, 39.3)
- moved JP16 1.77 mm to (73.5, 60.8)
- renumbered SW1 to CTRL
Routing:
- net 5V: track 276.4 -> 274.0 mm
- net DIRLS: track 73.9 -> 75.6 mm
- net OELS: track 71.7 -> 72.8 mm
Other:
- board size 99.2 x 52.8 mm -> 99.3 x 52.9 mm
- board text added: "5V"
- board text added: "5V DIRLS"
- board text added: "5V GND"
- board text added: "DIR-LS"
- board text added: "G1 GND"
- board text added: "GND"
- board text added: "GND 3V3"
- board text added: "GND 5V"
- board text added: "OE-LS"
