File: pcb/metrodisplay.kicad_pcb (KiCad board)
At the start: 2 copper layers, 99.3 x 52.9 mm, 31 parts, among them J1 USB_C_Receptacle_PowerOnly_6P, J2 Conn_02x08_Counter_Clockwise, J3 Screw_Terminal_01x02, U1 ESP32-DEVKITC, U3 SN74AHCT245PWR, U4 SN74AHCT245PWR

Commit message: Pong game!
Parts:
- removed CTRL: SW_Push, Connector_JST:JST_PH_B2B-PH-K_1x02_P2.00mm_Vertical
- added C21: C, easyeda2kicad:C1206, B.Cu at (60.3, 51.8)
- added C22: C, easyeda2kicad:C1206, B.Cu at (66.0, 51.8)
- added J10: Screw_Terminal_01x01, Connector_Wire:SolderWire-0.5sqmm_1x01_D0.9mm_OD2.1mm, F.Cu at (28.7, 57.6)
- added J11: Screw_Terminal_01x01, Connector_Wire:SolderWire-0.5sqmm_1x01_D0.9mm_OD2.1mm, F.Cu at (61.9, 65.6)
- added J12: Screw_Terminal_01x01, Connector_Wire:SolderWire-0.5sqmm_1x01_D0.9mm_OD2.1mm, F.Cu at (58.7, 65.6)
- added J13: Screw_Terminal_01x01, Connector_Wire:SolderWire-0.5sqmm_1x01_D0.9mm_OD2.1mm, F.Cu at (55.6, 65.6)
- added J14: Screw_Terminal_01x01, Connector_Wire:SolderWire-0.5sqmm_1x01_D0.9mm_OD2.1mm, F.Cu at (52.4, 65.6)
- added J15: Screw_Terminal_01x01, Connector_Wire:SolderWire-0.5sqmm_1x01_D0.9mm_OD2.1mm, F.Cu at (49.3, 65.6)
- added J4: Screw_Terminal_01x01, Connector_Wire:SolderWire-0.5sqmm_1x01_D0.9mm_OD2.1mm, F.Cu at (65.9, 57.6)
- added J6: Screw_Terminal_01x01, Connector_Wire:SolderWire-0.5sqmm_1x01_D0.9mm_OD2.1mm, F.Cu at (42.1, 65.6)
- added J7: Screw_Terminal_01x01, Connector_Wire:SolderWire-0.5sqmm_1x01_D0.9mm_OD2.1mm, F.Cu at (39.0, 65.6)
- added J8: Screw_Terminal_01x01, Connector_Wire:SolderWire-0.5sqmm_1x01_D0.9mm_OD2.1mm, F.Cu at (35.8, 65.6)
- added J9: Screw_Terminal_01x01, Connector_Wire:SolderWire-0.5sqmm_1x01_D0.9mm_OD2.1mm, F.Cu at (32.7, 65.6)
- added P1: R_US, Resistor_THT:R_Axial_DIN0204_L3.6mm_D1.6mm_P5.08mm_Horizontal, F.Cu at (40.2, 53.6)
- added R10: R_US, Resistor_THT:R_Axial_DIN0204_L3.6mm_D1.6mm_P5.08mm_Horizontal, F.Cu at (58.7, 57.6)
- added R11: R_US, Resistor_THT:R_Axial_DIN0204_L3.6mm_D1.6mm_P5.08mm_Horizontal, F.Cu at (55.6, 57.6)
- added R12: R_US, Resistor_THT:R_Axial_DIN0204_L3.6mm_D1.6mm_P5.08mm_Horizontal, F.Cu at (52.4, 57.6)
- added R13: R_US, Resistor_THT:R_Axial_DIN0204_L3.6mm_D1.6mm_P5.08mm_Horizontal, F.Cu at (49.3, 57.6)
- added R3: R_US, Resistor_THT:R_Axial_DIN0204_L3.6mm_D1.6mm_P5.08mm_Horizontal, F.Cu at (45.3, 57.6)
- added R4: R_US, Resistor_THT:R_Axial_DIN0204_L3.6mm_D1.6mm_P5.08mm_Horizontal, F.Cu at (42.1, 57.6)
- added R5: R_US, Resistor_THT:R_Axial_DIN0204_L3.6mm_D1.6mm_P5.08mm_Horizontal, F.Cu at (39.0, 57.6)
- added R6: R_US, Resistor_THT:R_Axial_DIN0204_L3.6mm_D1.6mm_P5.08mm_Horizontal, F.Cu at (35.8, 57.6)
- added R7: R_US, Resistor_THT:R_Axial_DIN0204_L3.6mm_D1.6mm_P5.08mm_Horizontal, F.Cu at (32.7, 57.6)
- added R8: R_US, Resistor_THT:R_Axial_DIN0204_L3.6mm_D1.6mm_P5.08mm_Horizontal, F.Cu at (54.3, 53.6)
- added R9: R_US, Resistor_THT:R_Axial_DIN0204_L3.6mm_D1.6mm_P5.08mm_Horizontal, F.Cu at (61.9, 57.6)
- added U: Screw_Terminal_01x01, Connector_Wire:SolderWire-0.5sqmm_1x01_D0.9mm_OD2.1mm, F.Cu at (45.3, 65.6)
Connections:
- U1 pad 1: unconnected-(U1-3V3-Pad1) -> 3V3
- U1 pad 23: CTRL -> unconnected-(U1-IO15-Pad23)
- U1 pad 3: unconnected-(U1-SENSOR_VP-Pad3) -> P1
- U1 pad 4: unconnected-(U1-SENSOR_VN-Pad4) -> P2
Routing:
- net CTRL: track 99.0 -> 0.00 mm
- net 3V3: track 0.00 -> 49.7 mm
- net P1: track 0.00 -> 42.0 mm
- net P2: track 0.00 -> 25.4 mm
- net OE: track 68.7 -> 72.6 mm
- net 5V: track 274.0 -> 277.5 mm
- net Net-(J11-Pin_1): track 0.00 -> 2.92 mm
- net Net-(J9-Pin_1): track 0.00 -> 2.92 mm
- net Net-(J8-Pin_1): track 0.00 -> 2.92 mm
- net Net-(J7-Pin_1): track 0.00 -> 2.92 mm
- net Net-(J6-Pin_1): track 0.00 -> 2.92 mm
- net Net-(J5-Pin_1): track 0.00 -> 2.92 mm
- net Net-(J15-Pin_1): track 0.00 -> 2.92 mm
- net Net-(J14-Pin_1): track 0.00 -> 2.92 mm
- net Net-(J13-Pin_1): track 0.00 -> 2.92 mm
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Other:
- board text added: "C"
- board text added: "D"
- board text added: "L"
- board text added: "P2"
- board text added: "R"
- board text added: "U"
